File: PCB/AMR_pcb/AMR_pcb.kicad_sch (KiCad schematic)
At the start: 0 parts

Commit message: updated docs with volt meter display
Parts:
- added C1, C2, C3, C4: 100n, symbol Device:C
- added C5: 10n, symbol Device:C
- added U1: STM32F401RETx, Package_QFP:LQFP-64_10x10mm_P0.5mm, symbol MCU_ST_STM32F4:STM32F401RETx
Connections:
- new net +3.3V: C1.1, C2.1, C3.1, C4.1, C5.1, U1.1 (VBAT), U1.19 (VDD), U1.32 (VDD), U1.48 (VDD), U1.64 (VDD)
- new net GND: C1.2, C2.2, C3.2, C4.2, C5.2, U1.12 (VSSA), U1.18 (VSS), U1.31 (VSS), U1.47 (VSS), U1.63 (VSS)
