Commit message: Tuning PI of AMR, and updated gazebo model

File: ros_ws/src/amr_description/urdf/base.xacro (robot description, xacro)
@@ -11,19 +11,13 @@
       </material>
     </visual>
-    <collision>
-      <origin xyz="${x} ${y} ${plate_thickness * 0.5 + pillar_height * 0.5}" rpy="0 0 0"/>
-      <geometry>
-        <box size="${pillar_size} ${pillar_size} ${pillar_height}"/>
-      </geometry>
-    </collision>
   </xacro:macro>
   <xacro:macro name="base_link">
-    <link name="base_footprint"/>
-    <joint name="base_footprint_joint" type="fixed">
-      <parent link="base_footprint"/>
-      <child link="base_link"/>
-      <origin xyz="0 0 ${base_clearance + (plate_thickness * 0.5)}" rpy="0 0 0"/>
+    <link name="base_link"/>
+    <joint name="chassis_joint" type="fixed">
+      <parent link="base_link"/>
+      <child link="chassis_link"/>
+      <origin xyz="0 0 ${chassis_z}" rpy="0 0 0"/>
     </joint>
-    <link name="base_link">
+    <link name="chassis_link">
       <!-- Bottom plate -->
       <visual>
@@ -36,10 +30,4 @@
         </material>
       </visual>
-      <collision>
-        <origin xyz="0 0 0" rpy="0 0 0"/>
-        <geometry>
-          <cylinder length="${plate_thickness}" radius="${base_collision_radius}"/>
-        </geometry>
-      </collision>
       <!-- Top plate -->
       <visual>
@@ -52,10 +40,12 @@
         </material>
       </visual>
-      <collision>
-        <origin xyz="0 0 ${pillar_height + plate_thickness}" rpy="0 0 0"/>
-        <geometry>
-          <cylinder length="${plate_thickness}" radius="${base_collision_radius}"/>
-        </geometry>
-      </collision>
+      <xacro:if value="${enable_base_collision}">
+        <collision>
+          <origin xyz="0 0 ${plate_thickness * 0.5 + pillar_height * 0.5}" rpy="0 0 0"/>
+          <geometry>
+            <box size="${plate_diameter} ${plate_diameter} ${base_height_total}"/>
+          </geometry>
+        </collision>
+      </xacro:if>
       <!-- Four pillars -->
       <xacro:pillar x="${ pillar_offset}" y="${ pillar_offset}"/>

File: ros_ws/src/amr_description/urdf/casters.xacro (robot description, xacro)
@@ -61,14 +61,10 @@
     </joint>
     <gazebo reference="front_caster_link">
-      <mu1>0.001</mu1>
-      <mu2>0.001</mu2>
-      <kp>10000.0</kp>
-      <kd>5.0</kd>
+      <mu1>${caster_mu1}</mu1>
+      <mu2>${caster_mu2}</mu2>
     </gazebo>
     <gazebo reference="rear_caster_link">
-      <mu1>0.001</mu1>
-      <mu2>0.001</mu2>
-      <kp>10000.0</kp>
-      <kd>5.0</kd>
+      <mu1>${caster_mu1}</mu1>
+      <mu2>${caster_mu2}</mu2>
     </gazebo>
   </xacro:macro>

File: ros_ws/src/amr_description/urdf/params.xacro (robot description, xacro)
@@ -2,25 +2,27 @@
 <robot xmlns:xacro="http://www.ros.org/wiki/xacro">
   <!-- Basic geometry (meters) -->
-  <xacro:property name="plate_diameter" value="0.40"/>
+  <xacro:property name="plate_diameter" value="0.386"/>
   <xacro:property name="plate_radius" value="${plate_diameter * 0.5}"/>
   <xacro:property name="plate_thickness" value="0.01"/>
   <xacro:property name="base_clearance" value="0.02"/>
   <xacro:property name="base_collision_clearance" value="0.02"/>
+  <xacro:property name="enable_base_collision" value="true"/>
   <xacro:property name="pillar_size" value="0.025"/>
   <xacro:property name="pillar_height" value="0.15"/>
-  <xacro:property name="pillar_offset" value="0.1"/>
+  <xacro:property name="pillar_offset" value="${plate_radius * 0.5}"/>
   <xacro:property name="total_mass" value="12.0"/>
   <xacro:property name="base_height_total" value="${(plate_thickness * 2.0) + pillar_height}"/>
-  <xacro:property name="wheel_radius" value="0.05"/>
+  <xacro:property name="wheel_radius" value="0.0615"/>
   <xacro:property name="wheel_width" value="0.025"/>
   <xacro:property name="wheel_mass" value="0.10"/>
-  <xacro:property name="track_width" value="${plate_diameter + wheel_width}"/>
+  <xacro:property name="track_width" value="0.386"/>
   <xacro:property name="wheel_y_offset" value="${track_width * 0.5}"/>
-  <xacro:property name="wheel_z" value="${wheel_radius - (base_clearance + (plate_thickness * 0.5))}"/>
+  <xacro:property name="wheel_z" value="0.0"/>
+  <xacro:property name="chassis_z" value="${(base_clearance + (plate_thickness * 0.5)) - wheel_radius}"/>
   <xacro:property name="base_collision_radius" value="${wheel_y_offset - wheel_radius - base_collision_clearance}"/>
   <xacro:property name="caster_radius" value="0.0127"/>
   <xacro:property name="caster_mass" value="0.05"/>
   <xacro:property name="caster_x_offset" value="${plate_radius - 0.02}"/>
-  <xacro:property name="caster_clearance" value="0.003"/>
+  <xacro:property name="caster_clearance" value="0.0"/>
   <xacro:property name="caster_z" value="${wheel_z - wheel_radius + caster_radius + caster_clearance}"/>
   <xacro:property name="lidar_height" value="0.05"/>
@@ -37,3 +39,11 @@
   <xacro:property name="camera_mass" value="0.10"/>
   <xacro:property name="base_mass" value="${total_mass - (2 * wheel_mass) - (2 * caster_mass) - lidar_mass - camera_mass}"/>
+  <!-- Gazebo friction tuning -->
+  <xacro:property name="wheel_mu1" value="1.0"/>
+  <xacro:property name="wheel_mu2" value="1.0"/>
+  <xacro:property name="wheel_slip1" value="0.0"/>
+  <xacro:property name="wheel_slip2" value="0.02"/>
+  <xacro:property name="wheel_fdir1" value="1 0 0"/>
+  <xacro:property name="caster_mu1" value="0.001"/>
+  <xacro:property name="caster_mu2" value="0.001"/>
 </robot>

File: ros_ws/src/amr_description/urdf/wheels.xacro (robot description, xacro)
@@ -66,18 +66,16 @@
     <!-- Gazebo surface parameters for wheel traction -->
     <gazebo reference="left_wheel_link">
-      <mu1>1.0</mu1>
-      <mu2>0.05</mu2>
-      <slip1>0.02</slip1>
-      <slip2>0.02</slip2>
-      <kp>100000.0</kp>
-      <kd>1.0</kd>
+      <mu1>${wheel_mu1}</mu1>
+      <mu2>${wheel_mu2}</mu2>
+      <fdir1>${wheel_fdir1}</fdir1>
+      <slip1>${wheel_slip1}</slip1>
+      <slip2>${wheel_slip2}</slip2>
     </gazebo>
     <gazebo reference="right_wheel_link">
-      <mu1>1.0</mu1>
-      <mu2>0.05</mu2>
-      <slip1>0.02</slip1>
-      <slip2>0.02</slip2>
-      <kp>100000.0</kp>
-      <kd>1.0</kd>
+      <mu1>${wheel_mu1}</mu1>
+      <mu2>${wheel_mu2}</mu2>
+      <fdir1>${wheel_fdir1}</fdir1>
+      <slip1>${wheel_slip1}</slip1>
+      <slip2>${wheel_slip2}</slip2>
     </gazebo>
   </xacro:macro>
