Commit message: Updated to basic gazebo simulation which responds to teleop

File: ros_ws/src/amr_description/urdf/amr.urdf.xacro (robot description, xacro)
@@ -1,289 +1,14 @@
 <?xml version="1.0"?>
 <robot name="amr" xmlns:xacro="http://www.ros.org/wiki/xacro">
-  <!-- Basic geometry (meters) -->
-  <xacro:property name="plate_diameter" value="0.40"/>
-  <xacro:property name="plate_radius" value="${plate_diameter * 0.5}"/>
-  <xacro:property name="plate_thickness" value="0.01"/>
-  <xacro:property name="pillar_size" value="0.025"/>
-  <xacro:property name="pillar_height" value="0.15"/>
-  <xacro:property name="pillar_offset" value="0.1"/>
-  <xacro:property name="total_mass" value="12.0"/>
-  <xacro:property name="base_height_total" value="${(plate_thickness * 2.0) + pillar_height}"/>
-  <xacro:property name="wheel_radius" value="0.05"/>
-  <xacro:property name="wheel_width" value="0.025"/>
-  <xacro:property name="wheel_mass" value="0.10"/>
-  <xacro:property name="wheel_y_offset" value="${plate_radius}"/>
-  <xacro:property name="wheel_z" value="${wheel_radius - (plate_thickness * 0.5)}"/>
-  <xacro:property name="caster_radius" value="0.0127"/>
-  <xacro:property name="caster_width" value="0.02"/>
-  <xacro:property name="caster_mass" value="0.05"/>
-  <xacro:property name="caster_x_offset" value="${plate_radius - 0.02}"/>
-  <xacro:property name="caster_z" value="${wheel_z - wheel_radius + caster_radius}"/>
-  <xacro:property name="lidar_height" value="0.05"/>
-  <xacro:property name="lidar_x" value="0.0"/>
-  <xacro:property name="lidar_y" value="0.0"/>
-  <xacro:property name="lidar_z" value="${pillar_height + (plate_thickness * 0.5) - (lidar_height * 0.5) + 0.05}"/>
-  <xacro:property name="camera_length" value="0.09"/>
-  <xacro:property name="camera_width" value="0.03"/>
-  <xacro:property name="camera_height" value="0.03"/>
-  <xacro:property name="camera_x" value="${plate_radius - (camera_length * 0.5)}"/>
-  <xacro:property name="camera_y" value="0.0"/>
-  <xacro:property name="camera_z" value="${pillar_height + plate_thickness + (camera_height * 0.5) + 0.05}"/>
-  <xacro:property name="lidar_mass" value="0.20"/>
-  <xacro:property name="camera_mass" value="0.10"/>
-  <xacro:property name="base_mass" value="${total_mass - (2 * wheel_mass) - (2 * caster_mass) - lidar_mass - camera_mass}"/>
-  <link name="base_footprint"/>
-  <joint name="base_footprint_joint" type="fixed">
-    <parent link="base_footprint"/>
-    <child link="base_link"/>
-    <origin xyz="0 0 ${plate_thickness * 0.5}" rpy="0 0 0"/>
-  </joint>
-  <link name="base_link">
-    <!-- Bottom plate -->
-    <visual>
-      <origin xyz="0 0 0.05" rpy="0 0 0"/>
-      <geometry>
-        <cylinder length="${plate_thickness}" radius="${plate_radius}"/>
-      </geometry>
-      <material name="gray">
-        <color rgba="0.6 0.6 0.6 1.0"/>
-      </material>
-    </visual>
-    <collision>
-      <origin xyz="0 0 0" rpy="0 0 0"/>
-      <geometry>
-        <cylinder length="${plate_thickness}" radius="${plate_radius}"/>
-      </geometry>
-    </collision>
-    <!-- Top plate -->
-    <visual>
-      <origin xyz="0 0 ${pillar_height + plate_thickness + 0.05}" rpy="0 0 0"/>
-      <geometry>
-        <cylinder length="${plate_thickness}" radius="${plate_radius}"/>
-      </geometry>
-      <material name="light_gray">
-        <color rgba="0.75 0.75 0.75 1.0"/>
-      </material>
-    </visual>
-    <collision>
-      <origin xyz="0 0 ${pillar_height + plate_thickness}" rpy="0 0 0"/>
-      <geometry>
-        <cylinder length="${plate_thickness}" radius="${plate_radius}"/>
-      </geometry>
-    </collision>
-    <!-- Four pillars -->
-    <xacro:macro name="pillar" params="x y">
-      <visual>
-        <origin xyz="${x} ${y} ${plate_thickness * 0.5 + pillar_height * 0.5 + 0.05}" rpy="0 0 0"/>
-        <geometry>
-          <box size="${pillar_size} ${pillar_size} ${pillar_height}"/>
-        </geometry>
-        <material name="dark_gray">
-          <color rgba="0.3 0.3 0.3 1.0"/>
-        </material>
-      </visual>
-      <collision>
-        <origin xyz="${x} ${y} ${plate_thickness * 0.5 + pillar_height * 0.5}" rpy="0 0 0"/>
-        <geometry>
-          <box size="${pillar_size} ${pillar_size} ${pillar_height}"/>
-        </geometry>
-      </collision>
-    </xacro:macro>
-    <xacro:pillar x="${ pillar_offset}" y="${ pillar_offset}"/>
-    <xacro:pillar x="${ pillar_offset}" y="${-pillar_offset}"/>
-    <xacro:pillar x="${-pillar_offset}" y="${ pillar_offset}"/>
-    <xacro:pillar x="${-pillar_offset}" y="${-pillar_offset}"/>
-    <inertial>
-      <origin xyz="0 0 ${base_height_total * 0.5}" rpy="0 0 0"/>
-      <mass value="${base_mass}"/>
-      <inertia
-        ixx="${(1.0/12.0) * base_mass * (3 * plate_radius * plate_radius + base_height_total * base_height_total)}"
-        iyy="${(1.0/12.0) * base_mass * (3 * plate_radius * plate_radius + base_height_total * base_height_total)}"
-        izz="${0.5 * base_mass * plate_radius * plate_radius}"
-        ixy="0.0" ixz="0.0" iyz="0.0"/>
-    </inertial>
-  </link>
-  <!-- Wheels -->
-  <link name="left_wheel_link">
-    <visual>
-      <origin xyz="0 0 0" rpy="1.5708 0 0"/>
-      <geometry>
-        <cylinder length="${wheel_width}" radius="${wheel_radius}"/>
-      </geometry>
-      <material name="black">
-        <color rgba="0.1 0.1 0.1 1.0"/>
-      </material>
-    </visual>
-    <collision>
-      <origin xyz="0 0 0" rpy="1.5708 0 0"/>
-      <geometry>
-        <cylinder length="${wheel_width}" radius="${wheel_radius}"/>
-      </geometry>
-    </collision>
-    <inertial>
-      <origin xyz="0 0 0" rpy="0 0 0"/>
-      <mass value="${wheel_mass}"/>
-      <inertia
-        ixx="${(1.0/12.0) * wheel_mass * (3 * wheel_radius * wheel_radius + wheel_width * wheel_width)}"
-        iyy="${0.5 * wheel_mass * wheel_radius * wheel_radius}"
-        izz="${(1.0/12.0) * wheel_mass * (3 * wheel_radius * wheel_radius + wheel_width * wheel_width)}"
-        ixy="0.0" ixz="0.0" iyz="0.0"/>
-    </inertial>
-  </link>
-  <link name="right_wheel_link">
-    <visual>
-      <origin xyz="0 0 0" rpy="1.5708 0 0"/>
-      <geometry>
-        <cylinder length="${wheel_width}" radius="${wheel_radius}"/>
-      </geometry>
-      <material name="black"/>
-    </visual>
-    <collision>
-      <origin xyz="0 0 0" rpy="1.5708 0 0"/>
-      <geometry>
-        <cylinder length="${wheel_width}" radius="${wheel_radius}"/>
-      </geometry>
-    </collision>
-    <inertial>
-      <origin xyz="0 0 0" rpy="0 0 0"/>
-      <mass value="${wheel_mass}"/>
-      <inertia
-        ixx="${(1.0/12.0) * wheel_mass * (3 * wheel_radius * wheel_radius + wheel_width * wheel_width)}"
-        iyy="${0.5 * wheel_mass * wheel_radius * wheel_radius}"
-        izz="${(1.0/12.0) * wheel_mass * (3 * wheel_radius * wheel_radius + wheel_width * wheel_width)}"
-        ixy="0.0" ixz="0.0" iyz="0.0"/>
-    </inertial>
-  </link>
-  <joint name="left_wheel_joint" type="continuous">
-    <parent link="base_link"/>
-    <child link="left_wheel_link"/>
-    <origin xyz="0 ${wheel_y_offset} ${wheel_z}" rpy="0 0 0"/>
-    <axis xyz="0 1 0"/>
-  </joint>
-  <joint name="right_wheel_joint" type="continuous">
-    <parent link="base_link"/>
-    <child link="right_wheel_link"/>
-    <origin xyz="0 ${-wheel_y_offset} ${wheel_z}" rpy="0 0 0"/>
-    <axis xyz="0 1 0"/>
-  </joint>
-  <!-- Casters (fixed for now) -->
-  <link name="front_caster_link">
-    <visual>
-      <origin xyz="0 0 0" rpy="1.5708 0 0"/>
-      <geometry>
-        <cylinder length="${caster_width}" radius="${caster_radius}"/>
-      </geometry>
-      <material name="black"/>
-    </visual>
-    <collision>
-      <origin xyz="0 0 0" rpy="1.5708 0 0"/>
-      <geometry>
-        <cylinder length="${caster_width}" radius="${caster_radius}"/>
-      </geometry>
-    </collision>
-    <inertial>
-      <origin xyz="0 0 0" rpy="0 0 0"/>
-      <mass value="${caster_mass}"/>
-      <inertia
-        ixx="${(1.0/12.0) * caster_mass * (3 * caster_radius * caster_radius + caster_width * caster_width)}"
-        iyy="${0.5 * caster_mass * caster_radius * caster_radius}"
-        izz="${(1.0/12.0) * caster_mass * (3 * caster_radius * caster_radius + caster_width * caster_width)}"
-        ixy="0.0" ixz="0.0" iyz="0.0"/>
-    </inertial>
-  </link>
-  <link name="rear_caster_link">
-    <visual>
-      <origin xyz="0 0 0" rpy="1.5708 0 0"/>
-      <geometry>
-        <cylinder length="${caster_width}" radius="${caster_radius}"/>
-      </geometry>
-      <material name="black"/>
-    </visual>
-    <collision>
-      <origin xyz="0 0 0" rpy="1.5708 0 0"/>
-      <geometry>
-        <cylinder length="${caster_width}" radius="${caster_radius}"/>
-      </geometry>
-    </collision>
-    <inertial>
-      <origin xyz="0 0 0" rpy="0 0 0"/>
-      <mass value="${caster_mass}"/>
-      <inertia
-        ixx="${(1.0/12.0) * caster_mass * (3 * caster_radius * caster_radius + caster_width * caster_width)}"
-        iyy="${0.5 * caster_mass * caster_radius * caster_radius}"
-        izz="${(1.0/12.0) * caster_mass * (3 * caster_radius * caster_radius + caster_width * caster_width)}"
-        ixy="0.0" ixz="0.0" iyz="0.0"/>
-    </inertial>
-  </link>
-  <joint name="front_caster_joint" type="fixed">
-    <parent link="base_link"/>
-    <child link="front_caster_link"/>
-    <origin xyz="${caster_x_offset} 0 ${caster_z}" rpy="0 0 0"/>
-  </joint>
-  <joint name="rear_caster_joint" type="fixed">
-    <parent link="base_link"/>
-    <child link="rear_caster_link"/>
-    <origin xyz="${-caster_x_offset} 0 ${caster_z}" rpy="0 0 0"/>
-  </joint>
-  <!-- Sensors -->
-  <link name="lidar_link">
-    <visual>
-      <origin xyz="0 0 0" rpy="0 0 0"/>
-      <geometry>
-        <cylinder length="${lidar_height}" radius="0.04"/>
-      </geometry>
-      <material name="black"/>
-    </visual>
-    <collision>
-      <origin xyz="0 0 0" rpy="0 0 0"/>
-      <geometry>
-        <cylinder length="${lidar_height}" radius="0.04"/>
-      </geometry>
-    </collision>
-    <inertial>
-      <origin xyz="0 0 0" rpy="0 0 0"/>
-      <mass value="${lidar_mass}"/>
-      <inertia
-        ixx="${(1.0/12.0) * lidar_mass * (3 * 0.04 * 0.04 + lidar_height * lidar_height)}"
-        iyy="${(1.0/12.0) * lidar_mass * (3 * 0.04 * 0.04 + lidar_height * lidar_height)}"
-        izz="${0.5 * lidar_mass * 0.04 * 0.04}"
-        ixy="0.0" ixz="0.0" iyz="0.0"/>
-    </inertial>
-  </link>
-  <joint name="lidar_joint" type="fixed">
-    <parent link="base_link"/>
-    <child link="lidar_link"/>
-    <origin xyz="${lidar_x} ${lidar_y} ${lidar_z}" rpy="3.14159 0 0"/>
-  </joint>
-  <link name="camera_link">
-    <visual>
-      <origin xyz="0 0 0" rpy="0 0 0"/>
-      <geometry>
-        <box size="${camera_length} ${camera_width} ${camera_height}"/>
-      </geometry>
-      <material name="blue">
-        <color rgba="0.2 0.2 0.8 1.0"/>
-      </material>
-    </visual>
-    <collision>
-      <origin xyz="0 0 0" rpy="0 0 0"/>
-      <geometry>
-        <box size="${camera_length} ${camera_width} ${camera_height}"/>
-      </geometry>
-    </collision>
-    <inertial>
-      <origin xyz="0 0 0" rpy="0 0 0"/>
-      <mass value="${camera_mass}"/>
-      <inertia
-        ixx="${(1.0/12.0) * camera_mass * (camera_width * camera_width + camera_height * camera_height)}"
-        iyy="${(1.0/12.0) * camera_mass * (camera_length * camera_length + camera_height * camera_height)}"
-        izz="${(1.0/12.0) * camera_mass * (camera_length * camera_length + camera_width * camera_width)}"
-        ixy="0.0" ixz="0.0" iyz="0.0"/>
-    </inertial>
-  </link>
-  <joint name="camera_joint" type="fixed">
-    <parent link="base_link"/>
-    <child link="camera_link"/>
-    <origin xyz="${camera_x} ${camera_y} ${camera_z}" rpy="0 0 0"/>
-  </joint>
+  <xacro:include filename="params.xacro"/>
+  <xacro:include filename="base.xacro"/>
+  <xacro:include filename="casters.xacro"/>
+  <xacro:include filename="wheels.xacro"/>
+  <xacro:include filename="sensors.xacro"/>
+  <xacro:include filename="ros2_control.xacro"/>
+  <xacro:base_link/>
+  <xacro:casters/>
+  <xacro:wheels/>
+  <xacro:sensors/>
+  <xacro:ros2_control_block/>
 </robot>

Commit message: Updated URDF + Gazebo model. Added ros2 control and updated dockerfile

File: ros_ws/src/amr_description/urdf/amr.urdf.xacro (robot description, xacro)
@@ -5,10 +5,12 @@
   <xacro:include filename="casters.xacro"/>
   <xacro:include filename="wheels.xacro"/>
-  <xacro:include filename="sensors.xacro"/>
+  <xacro:include filename="lidar.xacro"/>
+  <xacro:include filename="camera.xacro"/>
   <xacro:include filename="ros2_control.xacro"/>
   <xacro:base_link/>
   <xacro:casters/>
   <xacro:wheels/>
-  <xacro:sensors/>
+  <xacro:lidar_sensor/>
+  <xacro:camera_sensor/>
   <xacro:ros2_control_block/>
 </robot>

File: ros_ws/src/amr_description/urdf/base.xacro (robot description, xacro)
@@ -13,4 +13,10 @@
   </xacro:macro>
   <xacro:macro name="base_link">
+    <link name="base_footprint"/>
+    <joint name="base_footprint_joint" type="fixed">
+      <parent link="base_footprint"/>
+      <child link="base_link"/>
+      <origin xyz="0 0 ${wheel_radius}" rpy="0 0 0"/>
+    </joint>
     <link name="base_link"/>
     <joint name="chassis_joint" type="fixed">
@@ -42,7 +48,7 @@
       <xacro:if value="${enable_base_collision}">
         <collision>
-          <origin xyz="0 0 ${plate_thickness * 0.5 + pillar_height * 0.5}" rpy="0 0 0"/>
+          <origin xyz="0 0 0" rpy="0 0 0"/>
           <geometry>
-            <box size="${plate_diameter} ${plate_diameter} ${base_height_total}"/>
+            <cylinder length="${plate_thickness}" radius="${plate_radius}"/>
           </geometry>
         </collision>

File: ros_ws/src/amr_description/urdf/lidar.xacro (robot description, xacro)
@@ -1,5 +1,5 @@
 <?xml version="1.0"?>
 <robot xmlns:xacro="http://www.ros.org/wiki/xacro">
-  <xacro:macro name="sensors">
+  <xacro:macro name="lidar_sensor">
     <link name="lidar_link">
       <visual>
@@ -66,35 +66,4 @@
       </sensor>
     </gazebo>
-    <link name="camera_link">
-      <visual>
-        <origin xyz="0 0 0" rpy="0 0 0"/>
-        <geometry>
-          <box size="${camera_length} ${camera_width} ${camera_height}"/>
-        </geometry>
-        <material name="blue">
-          <color rgba="0.2 0.2 0.8 1.0"/>
-        </material>
-      </visual>
-      <collision>
-        <origin xyz="0 0 0" rpy="0 0 0"/>
-        <geometry>
-          <box size="${camera_length} ${camera_width} ${camera_height}"/>
-        </geometry>
-      </collision>
-      <inertial>
-        <origin xyz="0 0 0" rpy="0 0 0"/>
-        <mass value="${camera_mass}"/>
-        <inertia
-          ixx="${(1.0/12.0) * camera_mass * (camera_width * camera_width + camera_height * camera_height)}"
-          iyy="${(1.0/12.0) * camera_mass * (camera_length * camera_length + camera_height * camera_height)}"
-          izz="${(1.0/12.0) * camera_mass * (camera_length * camera_length + camera_width * camera_width)}"
-          ixy="0.0" ixz="0.0" iyz="0.0"/>
-      </inertial>
-    </link>
-    <joint name="camera_joint" type="fixed">
-      <parent link="base_link"/>
-      <child link="camera_link"/>
-      <origin xyz="${camera_x} ${camera_y} ${camera_z}" rpy="0 0 0"/>
-    </joint>
   </xacro:macro>
 </robot>

File: ros_ws/src/amr_description/urdf/params.xacro (robot description, xacro)
@@ -21,15 +21,17 @@
   <xacro:property name="chassis_z" value="${(base_clearance + (plate_thickness * 0.5)) - wheel_radius}"/>
   <xacro:property name="base_collision_radius" value="${wheel_y_offset - wheel_radius - base_collision_clearance}"/>
-  <xacro:property name="caster_radius" value="0.0127"/>
+  <xacro:property name="caster_radius" value="0.015"/>
   <xacro:property name="caster_mass" value="0.05"/>
   <xacro:property name="caster_x_offset" value="${plate_radius - 0.02}"/>
-  <xacro:property name="caster_clearance" value="0.0"/>
+  <xacro:property name="caster_clearance" value="0.001"/>
   <xacro:property name="caster_z" value="${wheel_z - wheel_radius + caster_radius + caster_clearance}"/>
   <xacro:property name="lidar_height" value="0.05"/>
   <xacro:property name="lidar_x" value="0.0"/>
   <xacro:property name="lidar_y" value="0.0"/>
-  <xacro:property name="lidar_z" value="${pillar_height + (plate_thickness * 0.5) - (lidar_height * 0.5)}"/>
-  <xacro:property name="camera_length" value="0.09"/>
-  <xacro:property name="camera_width" value="0.03"/>
+  <xacro:property name="lidar_gap" value="0.002"/>
+  <xacro:property name="lidar_raise" value="0.01"/>
+  <xacro:property name="lidar_z" value="${chassis_z + pillar_height + (plate_thickness * 0.5) - (lidar_height * 0.5) - lidar_gap + lidar_raise}"/>
+  <xacro:property name="camera_length" value="0.03"/>
+  <xacro:property name="camera_width" value="0.09"/>
   <xacro:property name="camera_height" value="0.03"/>
   <xacro:property name="camera_x" value="${plate_radius - (camera_length * 0.5)}"/>
@@ -40,10 +42,10 @@
   <xacro:property name="base_mass" value="${total_mass - (2 * wheel_mass) - (2 * caster_mass) - lidar_mass - camera_mass}"/>
   <!-- Gazebo friction tuning -->
-  <xacro:property name="wheel_mu1" value="1.0"/>
-  <xacro:property name="wheel_mu2" value="1.0"/>
+  <xacro:property name="wheel_mu1" value="10.0"/>
+  <xacro:property name="wheel_mu2" value="10.0"/>
   <xacro:property name="wheel_slip1" value="0.0"/>
-  <xacro:property name="wheel_slip2" value="0.02"/>
+  <xacro:property name="wheel_slip2" value="0.002"/>
   <xacro:property name="wheel_fdir1" value="1 0 0"/>
-  <xacro:property name="caster_mu1" value="0.001"/>
-  <xacro:property name="caster_mu2" value="0.001"/>
+  <xacro:property name="caster_mu1" value="0.02"/>
+  <xacro:property name="caster_mu2" value="0.02"/>
 </robot>

File: ros_ws/src/amr_description/urdf/ros2_control.xacro (robot description, xacro)
@@ -1,8 +1,20 @@
 <?xml version="1.0"?>
 <robot xmlns:xacro="http://www.ros.org/wiki/xacro">
+  <xacro:arg name="use_sim" default="true"/>
+  <xacro:arg name="left_cmd_topic" default="/amr/wheel_cmd_left"/>
+  <xacro:arg name="right_cmd_topic" default="/amr/wheel_cmd_right"/>
+  <xacro:arg name="state_topic" default="/amr/wheel_state"/>
   <xacro:macro name="ros2_control_block">
     <ros2_control name="amr_system" type="system">
       <hardware>
-        <plugin>gazebo_ros2_control/GazeboSystem</plugin>
+        <xacro:if value="$(arg use_sim)">
+          <plugin>gazebo_ros2_control/GazeboSystem</plugin>
+        </xacro:if>
+        <xacro:unless value="$(arg use_sim)">
+          <plugin>amr_hardware/AMRHardware</plugin>
+          <param name="left_cmd_topic">$(arg left_cmd_topic)</param>
+          <param name="right_cmd_topic">$(arg right_cmd_topic)</param>
+          <param name="state_topic">$(arg state_topic)</param>
+        </xacro:unless>
       </hardware>
       <joint name="left_wheel_joint">
@@ -17,9 +29,11 @@
       </joint>
     </ros2_control>
-    <gazebo>
-      <plugin name="gazebo_ros2_control" filename="libgazebo_ros2_control.so">
-        <parameters>$(optenv AMR_DESCRIPTION_SHARE)/config/ros2_control.yaml</parameters>
-      </plugin>
-    </gazebo>
+    <xacro:if value="$(arg use_sim)">
+      <gazebo>
+        <plugin name="gazebo_ros2_control" filename="libgazebo_ros2_control.so">
+          <parameters>$(optenv AMR_DESCRIPTION_SHARE)/config/ros2_control.yaml</parameters>
+        </plugin>
+      </gazebo>
+    </xacro:if>
   </xacro:macro>
 </robot>

File: ros_ws/src/amr_description/urdf/wheels.xacro (robot description, xacro)
@@ -68,14 +68,8 @@
       <mu1>${wheel_mu1}</mu1>
       <mu2>${wheel_mu2}</mu2>
-      <fdir1>${wheel_fdir1}</fdir1>
-      <slip1>${wheel_slip1}</slip1>
-      <slip2>${wheel_slip2}</slip2>
     </gazebo>
     <gazebo reference="right_wheel_link">
       <mu1>${wheel_mu1}</mu1>
       <mu2>${wheel_mu2}</mu2>
-      <fdir1>${wheel_fdir1}</fdir1>
-      <slip1>${wheel_slip1}</slip1>
-      <slip2>${wheel_slip2}</slip2>
     </gazebo>
   </xacro:macro>

Commit message: Add SO-101 AMR RViz description

File: ros_ws/src/amr_description/urdf/amr.urdf.xacro (robot description, xacro)
@@ -1,4 +1,11 @@
 <?xml version="1.0"?>
 <robot name="amr" xmlns:xacro="http://www.ros.org/wiki/xacro">
+  <xacro:arg name="enable_so101" default="false"/>
+  <xacro:arg name="so101_mount_x" default="0.14"/>
+  <xacro:arg name="so101_mount_y" default="0.00"/>
+  <xacro:arg name="so101_mount_z" default="0.125"/>
+  <xacro:arg name="so101_mount_roll" default="0.0"/>
+  <xacro:arg name="so101_mount_pitch" default="0.0"/>
+  <xacro:arg name="so101_mount_yaw" default="0.0"/>
   <xacro:include filename="params.xacro"/>
   <xacro:include filename="base.xacro"/>
@@ -7,4 +14,5 @@
   <xacro:include filename="lidar.xacro"/>
   <xacro:include filename="camera.xacro"/>
+  <xacro:include filename="so101.xacro"/>
   <xacro:include filename="ros2_control.xacro"/>
   <xacro:base_link/>
@@ -13,4 +21,10 @@
   <xacro:lidar_sensor/>
   <xacro:camera_sensor/>
+  <xacro:if value="$(arg enable_so101)">
+    <xacro:so101_arm
+      parent="base_link"
+      xyz="$(arg so101_mount_x) $(arg so101_mount_y) $(arg so101_mount_z)"
+      rpy="$(arg so101_mount_roll) $(arg so101_mount_pitch) $(arg so101_mount_yaw)"/>
+  </xacro:if>
   <xacro:ros2_control_block/>
 </robot>

File: ros_ws/src/amr_description/urdf/casters.xacro (robot description, xacro)
@@ -8,5 +8,7 @@
           <sphere radius="${caster_radius}"/>
         </geometry>
-        <material name="black"/>
+        <material name="black">
+          <color rgba="0.02 0.02 0.02 1.0"/>
+        </material>
       </visual>
       <collision>

File: ros_ws/src/amr_description/urdf/params.xacro (robot description, xacro)
@@ -40,5 +40,6 @@
   <xacro:property name="camera_x" value="${plate_radius - (camera_length * 0.5)}"/>
   <xacro:property name="camera_y" value="0.0"/>
-  <xacro:property name="camera_z" value="${pillar_height + (plate_thickness * 1.5) + (camera_height * 0.5)}"/>
+  <!-- AMR RealSense/depth camera sits on the lower plate, not the top plate. -->
+  <xacro:property name="camera_z" value="${chassis_z + (plate_thickness * 0.5) + (camera_height * 0.5)}"/>
   <xacro:property name="lidar_mass" value="0.20"/>
   <xacro:property name="camera_mass" value="0.10"/>
