Commit message: Record Orin SO-101 bringup checkpoint

File: ros_ws/src/amr_description/urdf/camera.xacro (robot description, xacro)
@@ -31,5 +31,5 @@
       <parent link="base_link"/>
       <child link="camera_link"/>
-      <origin xyz="${camera_x} ${camera_y} ${camera_z}" rpy="0 0 0"/>
+      <origin xyz="${camera_x} ${camera_y} ${camera_z}" rpy="${camera_roll} ${camera_pitch} ${camera_yaw}"/>
     </joint>
     <!-- Optical frame for correct image orientation (REP-103) -->

File: ros_ws/src/amr_description/urdf/params.xacro (robot description, xacro)
@@ -42,4 +42,8 @@
   <!-- AMR RealSense/depth camera sits on the lower plate, not the top plate. -->
   <xacro:property name="camera_z" value="${chassis_z + (plate_thickness * 0.5) + (camera_height * 0.5)}"/>
+  <!-- Physical D455 mount is inverted; keep camera TF aligned for depth/perception. -->
+  <xacro:property name="camera_roll" value="3.14159"/>
+  <xacro:property name="camera_pitch" value="0.0"/>
+  <xacro:property name="camera_yaw" value="0.0"/>
   <xacro:property name="lidar_mass" value="0.20"/>
   <xacro:property name="camera_mass" value="0.10"/>
